File: hardware/driver_board/driver_board.kicad_pcb (KiCad board)
At the start: 2 copper layers, 99 parts, among them J1 796949-2, J2 796949-2, J3 796949-2, J4 796949-2, J5 Adafruit_1979, Q1 Toshiba_TK4R3E06PL, Q2 Toshiba_TK4R3E06PL, Q3 Toshiba_TK4R3E06PL, Q4 Toshiba_TK4R3E06PL, Q5 Toshiba_TK4R3E06PL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

Commit message: update
Parts:
- moved R17 15.2 mm to (118.7, 107.3), turned to 180 degrees
- moved R20 15.2 mm to (126.4, 112.4), turned to 0 degrees
- moved D24 5.34 mm to (160.7, 156.5)
- moved R21 3.94 mm to (69.1, 107.4)
- moved D3 3.81 mm to (54.0, 127.6)
- moved D9 3.81 mm to (57.8, 127.6)
- moved U7 3.24 mm to (158.1, 83.8)
- moved J3 0.64 mm to (163.2, 70.5)
- moved U2 0.64 mm to (87.6, 150.5)
- moved R1 0.63 mm to (137.8, 150.5)
- moved R2 0.63 mm to (141.6, 150.5)
Routing:
- net +5V: track 0.00 -> 218.7 mm
- net +12V: track 0.00 -> 146.7 mm
- net Net-(C19-Pad1): track 0.00 -> 143.0 mm
- net GND: track 0.00 -> 128.8 mm
- net Net-(C18-Pad2): track 0.00 -> 107.0 mm
- net Net-(C16-Pad2): track 0.00 -> 101.7 mm
- net +3V3: track 0.00 -> 86.6 mm
- net Net-(C15-Pad2): track 0.00 -> 82.1 mm
- net Net-(R6-Pad1): track 0.00 -> 77.3 mm
- net Net-(R5-Pad1): track 0.00 -> 77.0 mm
- net +24V: track 0.00 -> 73.9 mm
- net Net-(C16-Pad1): track 0.00 -> 66.7 mm
- net Net-(C17-Pad2): track 0.00 -> 63.9 mm
- net Net-(C18-Pad1): track 0.00 -> 61.8 mm
- net Net-(D10-Pad2): track 0.00 -> 58.4 mm
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- added copper zone on F.Cu, net +3V3

Commit message: update PCB
Parts:
- moved D19 61.0 mm to (120.0, 94.0)
- moved Q7 61.0 mm to (120.0, 100.3)
- moved D17 61.0 mm to (108.6, 94.0)
- moved Q5 61.0 mm to (108.6, 100.3)
- moved D20 61.0 mm to (120.0, 81.3)
- moved Q8 61.0 mm to (120.0, 87.6)
- moved D18 61.0 mm to (108.6, 81.3)
- moved Q6 61.0 mm to (108.6, 87.6)
- moved F2 58.8 mm to (120.8, 67.1)
- moved J2 58.4 mm to (111.1, 70.5)
- moved C5 19.1 mm to (96.5, 101.6), turned to 90 degrees
- moved C3 18.7 mm to (83.8, 101.6), turned to 90 degrees
- moved C9 18.5 mm to (71.1, 101.6), turned to 90 degrees
- moved R22 13.1 mm to (69.2, 106.0), turned to 180 degrees
- moved C7 12.6 mm to (58.4, 101.6), turned to 90 degrees
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Connections:
- J3 pad 1: GND -> +24V
- J3 pad 2: +24V -> GND
Routing:
- net +24V: track 73.9 -> 202.2 mm
- net Net-(C15-Pad2): track 82.1 -> 193.4 mm
- net Net-(C17-Pad2): track 63.9 -> 161.3 mm, vias 0 -> 1
- net +12V: track 146.7 -> 207.6 mm
- net Net-(C18-Pad2): track 107.0 -> 162.5 mm, vias 0 -> 1
- net Net-(D12-Pad2): track 13.0 -> 64.3 mm, vias 0 -> 1
- net Net-(D9-Pad2): track 26.5 -> 74.8 mm
- net Net-(D11-Pad2): track 15.2 -> 61.5 mm, vias 0 -> 1
- net Net-(C16-Pad2): track 101.7 -> 138.4 mm
- net Net-(D10-Pad2): track 58.4 -> 91.7 mm
- net Net-(C17-Pad1): track 12.8 -> 43.4 mm
- net Net-(C18-Pad1): track 61.8 -> 41.2 mm
- net Net-(D7-Pad2): track 37.4 -> 45.2 mm
- net Net-(D6-Pad2): track 45.5 -> 53.0 mm, vias 0 -> 1
- net Net-(C15-Pad1): track 44.9 -> 52.3 mm
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
Commit message: update PCB
Parts:
- moved R17 6.35 mm to (118.7, 112.4)
- moved R18 6.35 mm to (103.5, 106.0)
Routing:
- net Net-(C15-Pad2): track 193.4 -> 158.7 mm
- net GND: track 125.9 -> 160.0 mm
- net Net-(D8-Pad2): track 42.3 -> 53.5 mm
- net Net-(D5-Pad2): track 55.9 -> 45.9 mm
- net Net-(D6-Pad2): track 53.0 -> 55.3 mm
- net Net-(D9-Pad2): track 74.8 -> 76.2 mm
- net Net-(D12-Pad2): track 64.3 -> 62.9 mm
- net Net-(D11-Pad2): track 61.5 -> 60.8 mm
- net Net-(C17-Pad2): track 161.3 -> 161.8 mm

Commit message: update PCB
Parts:
- added REF**: MountingHole_3.2mm_M3, MountingHole:MountingHole_3.2mm_M3, F.Cu at (196.6, 157.2)
- added REF**: MountingHole_3.2mm_M3, MountingHole:MountingHole_3.2mm_M3, F.Cu at (51.4, 156.8)
- added REF**: MountingHole_3.2mm_M3, MountingHole:MountingHole_3.2mm_M3, F.Cu at (196.6, 68.2)
- added REF**: MountingHole_3.2mm_M3, MountingHole:MountingHole_3.2mm_M3, F.Cu at (51.6, 68.2)
Routing:
- net Net-(C19-Pad1): track 143.5 -> 6.35 mm
- net GND: track 160.0 -> 282.8 mm
- net +24V: track 202.2 -> 83.7 mm
- net Net-(C16-Pad2): track 138.4 -> 96.1 mm
- net +5V: track 219.9 -> 183.0 mm
- net Net-(C18-Pad2): track 162.7 -> 132.5 mm
- net Net-(C17-Pad2): track 161.8 -> 145.2 mm
- net +12V: track 207.6 -> 191.2 mm
- net Net-(F2-Pad1): track 16.2 -> 0.00 mm
- net Net-(C15-Pad2): track 158.7 -> 145.1 mm
- net Net-(F1-Pad1): track 11.1 -> 0.00 mm
- net +3V3: track 86.6 -> 85.3 mm
- added copper zone on B.Cu, net +12V
- added copper zone on B.Cu, net +24V
- added copper zone on B.Cu, net +5V
- added copper zone on B.Cu, net GND
- added copper zone on F.Cu, net GND
- added copper zone on B.Cu, net Net-(C15-Pad2)
- added copper zone on B.Cu, net Net-(C16-Pad2)
- added copper zone on B.Cu, net Net-(C17-Pad2)
- added copper zone on B.Cu, net Net-(C18-Pad2)
- added copper zone on B.Cu, net Net-(C19-Pad1)
- added copper zone on B.Cu, net Net-(F1-Pad1)
- added copper zone on B.Cu, net Net-(F2-Pad1)
- removed copper zone on F.Cu, net +3V3
Other:
- board outline added: 155 x 100 mm
